File: pcb/power.kicad_sch (KiCad schematic)
At the start: 23 parts, among them J4 Conn_01x02, J5 ARM, Q1 PMOS, U10 LM3671MF, U11 TPS2116DRL

Commit message: Made terminal block smaller.
Parts:
- J5: footprint TerminalBlock_Phoenix:TerminalBlock_Phoenix_MKDS-3-2-5.08_1x02_P5.08mm_Horizontal -> TerminalBlock_Phoenix:TerminalBlock_Phoenix_MPT-0,5-2-2.54_1x02_P2.54mm_Horizontal; MP 1711026 -> 1725656
Changed lines of the file:
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@@
 			)
 		)
-		(property "Footprint" "TerminalBlock_Phoenix:TerminalBlock_Phoenix_MKDS-3-2-5.08_1x02_P5.08mm_Horizontal"
+		(property "Footprint" "TerminalBlock_Phoenix:TerminalBlock_Phoenix_MPT-0,5-2-2.54_1x02_P2.54mm_Horizontal"
 			(at 36.83 120.65 0)
 			(effects
@@
 			)
 		)
-		(property "Datasheet" "https://www.phoenixcontact.com/us/products/1711026/pdf"
+		(property "Datasheet" "https://www.phoenixcontact.com/us/products/1725656/pdf"
 			(at 36.83 120.65 0)
 			(effects
@@
 			)
 		)
-		(property "MP" "1711026"
+		(property "MP" "1725656"
 			(at 36.83 120.65 0)
 			(effects

Commit message: Removed DRC errors on schematic by adding power flags.
Changed lines of the file:
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@@
 	)
 	(junction
+		(at 86.36 59.69)
+		(diameter 0)
+		(color 0 0 0 0)
+	)
+	(junction
 		(at 153.67 72.39)
 		(diameter 0)
@@
 	(wire
 		(pts
-			(xy 83.82 59.69) (xy 88.9 59.69)
+			(xy 83.82 59.69) (xy 86.36 59.69)
 		)
 		(stroke
@@
 	(wire
 		(pts
+			(xy 86.36 59.69) (xy 88.9 59.69)
+		)
+		(stroke
+			(width 0)
+			(type default)
+		)
+	)
+	(wire
+		(pts
 			(xy 236.22 115.57) (xy 242.57 115.57)
 		)
@@
 					(unit 1)
 				)
+			)
+		)
+	)
+	(symbol
+		(lib_id "power:PWR_FLAG")
+		(at 86.36 59.69 0)
+		(unit 1)
+		(exclude_from_sim no)
+		(in_bom yes)
+		(on_board yes)
+		(dnp no)
+		(fields_autoplaced yes)
+		(property "Reference" "#FLG02"
+			(at 86.36 57.785 0)
+			(effects
+				(font
+					(size 1.27 1.27)
+				)
+				(hide yes)
+			)
+		)
+		(property "Value" "~"
+			(at 86.36 55.88 0)
+			(effects
+				(font
+					(size 1.27 1.27)
+				)
+			)
+		)
+		(property "Footprint" ""
+			(at 86.36 59.69 0)
+			(effects
+				(font
+					(size 1.27 1.27)
+				)
+				(hide yes)
+			)
+		)
+		(property "Datasheet" "~"
+			(at 86.36 59.69 0)
+			(effects
+				(font
+					(size 1.27 1.27)
+				)
+				(hide yes)
+			)
+		)
+		(property "Description" "Special symbol for telling ERC where power comes from"
+			(at 86.36 59.69 0)
+			(effects
+				(font
+					(size 1.27 1.27)
+				)
+				(hide yes)
+			)
+		)
+		(pin "1"
+		)
+		(instances
+			(project ""
+				(path "/b90d3133-97a4-4747-8a68-e80f353c7b97/8d42d8f3-e666-4352-a3e9-99ac4271efe0"
+					(reference "#FLG02")
+					(unit 1)
+				)
