File: pcb/radio.kicad_sch (KiCad schematic)
At the start: 5 parts, among them J3 SMA_Coax, U11 RN2903

Commit message: Filled out the BOM for the schematic. Consolidated some components and changed footprint sizes.
Parts:
- C25, C26: footprint Capacitor_SMD:C_0201_0603Metric -> Capacitor_SMD:C_0402_1005Metric; MP (none) -> GRM155R61A104KA01J
- C27: value 2u2 -> 4u7; MP (none) -> CGA3E1X5R0J475K080AC
- J3: MP (none) -> 2484637-1
- U9: renamed from U11; MP RN2903-I/RM095 -> RN2903A-I/RMSA103
Changed lines of the file:
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@@
 			)
 		)
-		(property "Value" "2u2"
+		(property "Value" "4u7"
 			(at 208.28 81.2799 0)
 			(effects
@@
 			)
 		)
-		(property "Datasheet" "~"
+		(property "Datasheet" "https://product.tdk.com/system/files/dam/doc/product/capacitor/ceramic/mlcc/catalog/mlcc_automotive_general_en.pdf?ref_disty=mouser"
 			(at 204.47 80.01 0)
 			(effects
@@
 		)
 		(property "Description" "Unpolarized capacitor"
+			(at 204.47 80.01 0)
+			(effects
+				(font
+					(size 1.27 1.27)
+				)
+				(hide yes)
+			)
+		)
+		(property "MP" "CGA3E1X5R0J475K080AC"
 			(at 204.47 80.01 0)
 			(effects
@@
 			)
 		)
-		(property "Footprint" "Capacitor_SMD:C_0201_0603Metric"
+		(property "Footprint" "Capacitor_SMD:C_0402_1005Metric"
 			(at 178.7652 83.82 0)
 			(effects
@@
 			)
 		)
-		(property "Datasheet" "~"
+		(property "Datasheet" "https://www.mouser.ca/datasheet/2/281/1/GRM155R61A104KA01_02A-1983866.pdf"
 			(at 177.8 80.01 0)
 			(effects
@@
 		)
 		(property "Description" "Unpolarized capacitor"
+			(at 177.8 80.01 0)
+			(effects
+				(font
+					(size 1.27 1.27)
+				)
+				(hide yes)
+			)
+		)
+		(property "MP" "GRM155R61A104KA01J "
 			(at 177.8 80.01 0)
 			(effects
@@
 		(dnp no)
 		(fields_autoplaced yes)
-		(property "Reference" "U11"
+		(property "Reference" "U9"
 			(at 147.32 77.47 0)
 			(effects
@@
 			)
 		)
-		(property "Datasheet" ""
+		(property "Datasheet" "https://www.mouser.ca/datasheet/2/268/RN2903_Low_Power_Long_Range_LoRa_Technology_Transc-3444753.pdf"
 			(at 147.32 107.95 0)
 			(effects
@@
 			)
 		)
-		(property "MP" "RN2903-I/RM095"
+		(property "MP" "RN2903A-I/RMSA103"
 			(at 147.32 107.95 0)
 			(effects
@@
 			(project ""
 				(path "/b90d3133-97a4-4747-8a68-e80f353c7b97/4aee52ff-1633-42f1-aa90-3806408b7a97"
-					(reference "U11")
+					(reference "U9")
 					(unit 1)
 				)
@@
 			)
 		)
-		(property "Datasheet" "~"
+		(property "Datasheet" "https://www.mouser.ca/datasheet/2/418/9/ENG_CD_2484637_A-3480023.pdf"
 			(at 179.07 97.79 0)
 			(effects
@@
 		)
 		(property "Description" "small coaxial connector (BNC, SMA, SMB, SMC, Cinch/RCA, LEMO, ...)"
+			(at 179.07 97.79 0)
+			(effects
+				(font
+					(size 1.27 1.27)
+				)
+				(hide yes)
+			)
+		)
+		(property "MP" "2484637-1"
 			(at 179.07 97.79 0)
 			(effects
@@
 			)
 		)
-		(property "Footprint" "Capacitor_SMD:C_0201_0603Metric"
+		(property "Footprint" "Capacitor_SMD:C_0402_1005Metric"
 			(at 191.4652 83.82 0)
 			(effects
@@
 			)
 		)
-		(property "Datasheet" "~"
+		(property "Datasheet" "https://www.mouser.ca/datasheet/2/281/1/GRM155R61A104KA01_02A-1983866.pdf"
 			(at 190.5 80.01 0)
 			(effects
@@
 			(at 190.5 80.01 0)
 			(effects
+				(font
+					(size 1.27 1.27)
+				)
+				(hide yes)
+			)
+		)
+		(property "MP" "GRM155R61A104KA01J "
+			(at 190.5 80.01 0)
+			(effects

Commit message: Removed DRC errors on schematic by adding power flags.
Connections:
- no-connect marks 19 -> 20
Changed lines of the file:
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@@
+	)
+	(no_connect
+		(at 127 97.79)
 	)
 	(no_connect
