File: flight-computer/power.kicad_sch (KiCad schematic)
At the start: 23 parts, among them J4 Conn_01x02, J5 ARM, Q1 PMOS, U10 LM3671MF, U11 TPS2116DRL

Commit message: Remove out of stock LED from BOMS
Parts:
- D4: MP LG R971-KN-1 -> HSMG-C170
Changed lines of the file:
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@@
 			)
 		)
-		(property "Datasheet" "https://www.mouser.ca/datasheet/2/588/prd_pim_datasheet_2191277_EN_pdf-3419125.pdf"
+		(property "Datasheet" ""
 			(at 92.71 114.3 0)
 			(effects
@@
 			)
 		)
-		(property "MP" "LG R971-KN-1"
+		(property "MP" "HSMG-C170"
 			(at 92.71 114.3 0)
 			(effects
